File: EE514 Project/EE514 Project.sch (KiCad schematic (older format))
At the start: 0 parts

Commit message: Started schematic
Parts:
- added C? (x3): 10pF, symbol Device:C
- added C? (x3): 0.1uF, symbol Device:C
- added J?: Conn_01x03, symbol Connector_Generic:Conn_01x03
- added JP? (x2): Jumper_2_Bridged, symbol Jumper:Jumper_2_Bridged
- added R?: 10k, symbol Device:R_US
- added TP?: TestPoint, symbol Connector:TestPoint
- added U?: ADF411x, Package_SO:TSSOP-16_4.4x5mm_P0.65mm, symbol EE514_Board:ADF411x
- added U?: Teensy-LC, symbol teensy:Teensy-LC
Connections:
- new net: R?.1, U?.1 (FLo)
- new net: JP?.2 (B), U?.10 (CE)
- new net: C?.1, C?.1, JP?.2 (B), TP?.1, U?.16 (VP)
- new net +5V: C?.1, C?.1, C?.1, C?.1, JP?.1 (A), JP?.1 (A), U?.15 (DVDD), U?.7 (AVDD)
- new net CLK_PLL: J?.1 (Pin_1), U?.11 (CLK), U?.21 (14_A0_SCK0)
- new net DATA_PLL: J?.2 (Pin_2), U?.12 (DATA), U?.13 (11_MOSI0)
- new net GND: C?.2, C?.2, C?.2, C?.2, C?.2, C?.2, R?.2, U?.1 (GND), U?.17 (GND), U?.3 (CPGND), U?.32 (GND), U?.4 (AGND), U?.9 (DGND)
- new net LE_PLL: J?.3 (Pin_3), U?.12 (10_TX2_CS0_PWM), U?.13 (LE)
- new net Reference Oscillator/10MHz_REF_OUT: U?.8 (REFIN)
Other:
- note added: "Cut JP to externally \npower chargepumps"

Commit message: Finished layout and generated gerbers
Parts:
- removed U?: Teensy-LC, symbol teensy:Teensy-LC
- added C107, C110: 30pF, EE514 Board:C_0603_1608Metric_Pad0.98x0.95mm_HandSolder, symbol Device:C
- added C108: 56pF, EE514 Board:C_0603_1608Metric_Pad0.98x0.95mm_HandSolder, symbol Device:C
- added C109: 1.3nF, EE514 Board:C_0603_1608Metric_Pad0.98x0.95mm_HandSolder, symbol Device:C
- added D101, D102: LED, irex_LED_SMD:LED_Kingbright_AA3528V_3.5x2.8mm_handsolder, symbol Device:LED
- added H101, H102, H103, H104: MountingHole_Pad, MountingHole:MountingHole_2.2mm_M2_Pad_Via, symbol Mechanical:MountingHole_Pad
- added J101: Screw_Terminal_01x02, TerminalBlock_TE-Connectivity:TerminalBlock_TE_282834-2_1x02_P2.54mm_Horizontal, symbol Connector:Screw_Terminal_01x02
- added J103: SMA, Connector_Coaxial:SMA_Molex_73251-1153_EdgeMount_Horizontal, symbol Connector:Conn_Coaxial
- added R101, R102: 1k, EE514 Board:R_0603_1608Metric_Pad0.98x0.95mm_HandSolder, symbol Device:R_US
- added R104: 46.9k, EE514 Board:R_0603_1608Metric_Pad0.98x0.95mm_HandSolder, symbol Device:R_US
- added R105: 220k, EE514 Board:R_0603_1608Metric_Pad0.98x0.95mm_HandSolder, symbol Device:R_US
- added R106: 51, EE514 Board:R_0603_1608Metric_Pad0.98x0.95mm_HandSolder, symbol Device:R_US
- added TP101: TestPoint, TestPoint:TestPoint_THTPad_D1.5mm_Drill0.7mm, symbol Connector:TestPoint
- C101, C103, C106: renamed from C?; footprint (none) -> EE514 Board:C_0603_1608Metric_Pad0.98x0.95mm_HandSolder; Digi-Key PN (none) -> 399-C0603C104Z3VAC7867CT-ND
- C102, C104, C105: renamed from C?; footprint (none) -> EE514 Board:C_0603_1608Metric_Pad0.98x0.95mm_HandSolder; Digi-Key PN (none) -> 399-C0603C100J3HAC7867CT-ND
- J102: renamed from J?; value Conn_01x03 -> Conn_01x04; footprint (none) -> Connector_PinHeader_2.54mm:PinHeader_1x04_P2.54mm_Vertical; symbol Connector_Generic:Conn_01x03 -> Connector_Generic:Conn_01x04; Digi-Key PN (none) -> 732-5316-ND
- JP101, JP102: renamed from JP?; footprint (none) -> Jumper:SolderJumper-2_P1.3mm_Bridged2Bar_RoundedPad1.0x1.5mm
- R103: renamed from R?; footprint (none) -> EE514 Board:R_0603_1608Metric_Pad0.98x0.95mm_HandSolder; Digi-Key PN (none) -> 311-10.0KHRCT-ND
- TP102: renamed from TP?; footprint (none) -> TestPoint:TestPoint_THTPad_D1.5mm_Drill0.7mm
- U101: renamed from U?; value ADF411x -> ADF4117; Digi-Key PN (none) -> ADF4117BRUZ-RL7CT-ND
Connections:
- net +5V: now also J101.1 (Pin_1), R101.2
- net CLK_PLL: now also J102.2 (Pin_2); no longer J102.1 (Pin_1)
- net DATA_PLL: now also J102.3 (Pin_3); no longer J102.2 (Pin_2)
- net GND: now also J102.1 (Pin_1), C107.2, C108.2, C109.2, D101.1 (K), D102.1 (K), H101.1, H102.1, H103.1, H104.1, J101.2 (Pin_2), J103.2 (Ext), R106.2
- net LE_PLL: now also J102.4 (Pin_4); no longer J102.3 (Pin_3)
- net LOCKED: now reaches U101.14 (MUXOUT)
- net LOCKED: now also R102.2
- net Vp: now reaches C105.1, C106.1, JP102.2 (B), TP102.1, U101.16 (VP)
- net CP_OUT: now reaches U101.2 (CP)
- net CP_OUT: now also C108.1, R104.1, R105.2
- net at U101.5 (RFIN_B): now also C107.1
- net at U101.6 (RFIN_A): now also C110.2
- new net: D102.2 (A), R102.1, TP101.1
- new net: C109.1, R104.2
- new net: D101.2 (A), R101.1
- new net RF_OUT: C110.1, J103.1 (In), R106.1
- new net V_TUNE: R105.1
Other:
- note added: "Lock Indicator"
- note added: "Mounting Holes"
- note added: "Power Input"
- note added: "VCO input capacitance ~~5pF"
- moved on the sheet: C101, C102, C103, C104, C105, C106, JP101, JP102, R103, TP102, U101
