File: EE514 Project/EE514 Project.kicad_pcb (KiCad board)
At the start: 4 copper layers, 46.2 x 33.5 mm, 60 parts, among them J101 Screw_Terminal_01x02, J102 Conn_01x04, J103 SMA, Q301 BFP620, U101 ADF4117, U201 NC7SZ04, U401 TLC2201

Commit message: Added DC blocking cap to ref in
Parts:
- added C111: 1.3nF, EE514 Board:C_0603_1608Metric_Pad0.98x0.95mm_HandSolder, F.Cu at (146.1, 112.5)
Connections:
- U101 pad 8: /Reference Oscillator/10MHz_REF_OUT -> Net-(C111-Pad1)
Routing:
- net /Reference Oscillator/10MHz_REF_OUT: track 25.1 -> 20.3 mm
- net Net-(C111-Pad1): track 0.00 -> 2.26 mm
Changed lines of the file:
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@@
     (thickness 1.6)
     (drawings 67)
-    (tracks 260)
+    (tracks 262)
     (zones 0)
-    (modules 60)
-    (nets 35)
+    (modules 61)
+    (nets 36)
   )
   (page A4)
@@
   (net 33 /RF_OUT)
   (net 34 /V_TUNE)
+  (net 35 "Net-(C111-Pad1)")
   (net_class Default "This is the default net class."
     (clearance 0.2)
@@
     (add_net "Net-(C109-Pad1)")
     (add_net "Net-(C110-Pad2)")
+    (add_net "Net-(C111-Pad1)")
     (add_net "Net-(C201-Pad1)")
     (add_net "Net-(C301-Pad1)")
@@
     (add_net "Net-(U401-Pad5)")
     (add_net "Net-(U401-Pad8)")
+  )
+  (module "EE514 Board:C_0603_1608Metric_Pad0.98x0.95mm_HandSolder" (layer F.Cu)
+    (at 146.05 112.522 180)
+    (fp_text reference C111 (at 0 -1.27) (layer F.SilkS)
+      (effects (font (size 0.8128 0.8128) (thickness 0.15)))
+    )
+    (fp_text value 1.3nF (at 0.0254 2.1082) (layer F.Fab)
+      (effects (font (size 1 1) (thickness 0.15)))
+    )
+    (fp_text user %R (at 0 0) (layer F.Fab)
+      (effects (font (size 0.4 0.4) (thickness 0.06)))
+    )
+    (fp_line (start 0.8 0.4125) (end -0.8 0.4125) (layer F.Fab) (width 0.1))
+    (fp_line (start -0.254724 -0.5225) (end 0.254724 -0.5225) (layer F.SilkS) (width 0.12))
+    (fp_line (start -0.8 -0.4125) (end 0.8 -0.4125) (layer F.Fab) (width 0.1))
+    (fp_line (start -0.8 0.4125) (end -0.8 -0.4125) (layer F.Fab) (width 0.1))
+    (fp_line (start 0.8 -0.4125) (end 0.8 0.4125) (layer F.Fab) (width 0.1))
+    (fp_line (start -1.65 0.73) (end -1.65 -0.73) (layer F.CrtYd) (width 0.05))
+    (fp_line (start -1.65 -0.73) (end 1.65 -0.73) (layer F.CrtYd) (width 0.05))
+    (fp_line (start 1.65 -0.73) (end 1.65 0.73) (layer F.CrtYd) (width 0.05))
+    (fp_line (start 1.65 0.73) (end -1.65 0.73) (layer F.CrtYd) (width 0.05))
+    (fp_line (start -0.254724 0.5225) (end 0.254724 0.5225) (layer F.SilkS) (width 0.12))
+    (pad 2 smd rect (at 0.9125 0 180) (size 0.975 0.95) (layers F.Cu F.Paste F.Mask)
+      (net 26 "/Reference Oscillator/10MHz_REF_OUT"))
+    (pad 1 smd rect (at -0.9125 0 180) (size 0.975 0.95) (layers F.Cu F.Paste F.Mask)
+      (net 35 "Net-(C111-Pad1)"))
+    (model ${KISYS3DMOD}/Capacitor_SMD.3dshapes/C_0603_1608Metric.wrl
+      (at (xyz 0 0 0))
+      (scale (xyz 1 1 1))
+      (rotate (xyz 0 0 0))
+    )
+  )
+  (module irex_LED_SMD:LED_Kingbright_AA3528V_3.5x2.8mm_handsolder (layer F.Cu)
+    (at 165.227 117.856 90)
+    (descr "Pink SMD LED, 20mA, Kingbright")
+    (tags "SMD LED Kingbright ")
+    (attr smd)
+    (fp_text reference D102 (at -2.54 0 180) (layer F.SilkS)
+      (effects (font (size 0.8128 0.8128) (thickness 0.15)))
+    )
+    (fp_text value LED (at 2.1 3 90) (layer F.Fab)
+      (effects (font (size 1 1) (thickness 0.15)))
+    )
+    (fp_line (start 2.1 -1.779954) (end -1.4 -1.779954) (layer F.SilkS) (width 0.12))
+    (fp_line (start -1.4 -1.779954) (end -1.4 1.779954) (layer F.SilkS) (width 0.12))
+    (fp_line (start -1.4 1.779954) (end 2.1 1.779954) (layer F.SilkS) (width 0.12))
+    (fp_line (start 4.85 1.65) (end -1.25 1.65) (layer F.CrtYd) (width 0.05))
+    (fp_line (start -1.25 1.65) (end -1.25 -1.65) (layer F.CrtYd) (width 0.05))
+    (fp_line (start -1.25 -1.65) (end 4.85 -1.65) (layer F.CrtYd) (width 0.05))
+    (fp_line (start 4.85 -1.65) (end 4.85 1.65) (layer F.CrtYd) (width 0.05))
+    (fp_line (start 0.907106 -1.4) (end 3.4 -1.4) (layer F.Fab) (width 0.1))
+    (fp_line (start 3.4 -1.4) (end 3.4 1.4) (layer F.Fab) (width 0.1))
+    (fp_line (start 3.4 1.4) (end 0.199999 1.399999) (layer F.Fab) (width 0.1))
+    (fp_line (start 0.199999 1.399999) (end 0.199999 -0.692893) (layer F.Fab) (width 0.1))
+    (fp_line (start 0.199999 -0.692893) (end 0.907106 -1.4) (layer F.Fab) (width 0.1))
+    (pad 2 smd rect (at 3.6 0.01 90) (size 2 2.2) (layers F.Cu F.Paste F.Mask)
+      (net 17 "Net-(D102-Pad2)"))
+    (pad 1 smd roundrect (at 0 0.01 90) (size 2 2.2) (layers F.Cu F.Paste F.Mask) (roundrect_rratio 0.1)
+      (net 1 GND))
+    (model ${KICAD_IREX_3DMOD}/irex_LED_SMD.3dshapes/LED_Kingsbright_AA3528V_3.5x2.8mm_handsolder.step
+      (at (xyz 0 0 0))
+      (scale (xyz 1 1 1))
+      (rotate (xyz 0 0 0))
+    )
   )
   (module Connector_PinHeader_2.54mm:PinHeader_1x04_P2.54mm_Vertical (layer F.Cu)
@@
     (tags "TSSOP SO")
     (attr smd)
-    (fp_text reference U101 (at 0 3.556 90) (layer F.SilkS)
+    (fp_text reference U101 (at 2.286 3.302 90) (layer F.SilkS)
       (effects (font (size 0.8128 0.8128) (thickness 0.15)))
     )
@@
       (net 1 GND))
     (pad 8 smd roundrect (at -2.8625 2.275 270) (size 1.475 0.4) (layers F.Cu F.Paste F.Mask) (roundrect_rratio 0.25)
-      (net 26 "/Reference Oscillator/10MHz_REF_OUT"))
+      (net 35 "Net-(C111-Pad1)"))
     (pad 7 smd roundrect (at -2.8625 1.625 270) (size 1.475 0.4) (layers F.Cu F.Paste F.Mask) (roundrect_rratio 0.25)
       (net 2 +5V))
@@
     (descr "Potentiometer, horizontal, Bourns PV36W, https://www.bourns.com/docs/Product-Datasheets/pv36.pdf")
     (tags "Potentiometer horizontal Bourns PV36W")
-    (fp_text reference RV201 (at 3.556 0 270) (layer F.SilkS)
+    (fp_text reference RV201 (at 3.302 2.794 270) (layer F.SilkS)
       (effects (font (size 0.8128 0.8128) (thickness 0.15)))
     )
@@
       (net 1 GND))
     (model ${KISYS3DMOD}/Diode_SMD.3dshapes/D_SOD-523.wrl
-      (at (xyz 0 0 0))
-      (scale (xyz 1 1 1))
-      (rotate (xyz 0 0 0))
-    )
-  )
-  (module irex_LED_SMD:LED_Kingbright_AA3528V_3.5x2.8mm_handsolder (layer F.Cu)
-    (at 165.227 117.856 90)
-    (descr "Pink SMD LED, 20mA, Kingbright")
-    (tags "SMD LED Kingbright ")
-    (attr smd)
-    (fp_text reference D102 (at -2.54 0 180) (layer F.SilkS)
-      (effects (font (size 0.8128 0.8128) (thickness 0.15)))
-    )
-    (fp_text value LED (at 2.1 3 90) (layer F.Fab)
-      (effects (font (size 1 1) (thickness 0.15)))
-    )
-    (fp_line (start 0.199999 -0.692893) (end 0.907106 -1.4) (layer F.Fab) (width 0.1))
-    (fp_line (start 0.199999 1.399999) (end 0.199999 -0.692893) (layer F.Fab) (width 0.1))
-    (fp_line (start 3.4 1.4) (end 0.199999 1.399999) (layer F.Fab) (width 0.1))
-    (fp_line (start 3.4 -1.4) (end 3.4 1.4) (layer F.Fab) (width 0.1))
-    (fp_line (start 0.907106 -1.4) (end 3.4 -1.4) (layer F.Fab) (width 0.1))
-    (fp_line (start 4.85 -1.65) (end 4.85 1.65) (layer F.CrtYd) (width 0.05))
-    (fp_line (start -1.25 -1.65) (end 4.85 -1.65) (layer F.CrtYd) (width 0.05))
-    (fp_line (start -1.25 1.65) (end -1.25 -1.65) (layer F.CrtYd) (width 0.05))
-    (fp_line (start 4.85 1.65) (end -1.25 1.65) (layer F.CrtYd) (width 0.05))
-    (fp_line (start -1.2 1.779954) (end 2.3 1.779954) (layer F.SilkS) (width 0.12))
-    (fp_line (start -1.2 -1.779954) (end -1.2 1.779954) (layer F.SilkS) (width 0.12))
-    (fp_line (start 2.3 -1.779954) (end -1.2 -1.779954) (layer F.SilkS) (width 0.12))
-    (pad 2 smd rect (at 3.6 0.01 90) (size 2 2.2) (layers F.Cu F.Paste F.Mask)
-      (net 17 "Net-(D102-Pad2)"))
-    (pad 1 smd roundrect (at 0 0.01 90) (size 2 2.2) (layers F.Cu F.Paste F.Mask) (roundrect_rratio 0.1)
-      (net 1 GND))
-    (model ${KICAD_IREX_3DMOD}/irex_LED_SMD.3dshapes/LED_Kingsbright_AA3528V_3.5x2.8mm_handsolder.step
       (at (xyz 0 0 0))
       (scale (xyz 1 1 1))
@@
   (segment (start 137.407 117.592) (end 140.472 117.592) (width 0.3048) (layer F.Cu) (net 26))
   (segment (start 141.478 114.046) (end 141.478 116.586) (width 0.3048) (layer F.Cu) (net 26))
-  (segment (start 148.5425 111.379) (end 148.601 111.4375) (width 0.3048) (layer F.Cu) (net 26))
+  (segment (start 148.5425 111.379) (end 148.601 111.4375) (width 0.3048) (layer F.Cu) (net 35))
   (segment (start 142.875 117.983) (end 141.478 116.586) (width 0.3048) (layer F.Cu) (net 26))
   (segment (start 142.875 123.063) (end 142.875 117.983) (width 0.3048) (layer F.Cu) (net 26))
   (segment (start 141.478 124.46) (end 142.875 123.063) (width 0.3048) (layer F.Cu) (net 26))
-  (segment (start 141.478 114.046) (end 141.478 112.776) (width 0.3048) (layer F.Cu) (net 26))
-  (segment (start 142.8165 111.4375) (end 148.601 111.4375) (width 0.3048) (layer F.Cu) (net 26))
-  (segment (start 141.478 112.776) (end 142.8165 111.4375) (width 0.3048) (layer F.Cu) (net 26))
+  (segment (start 143.002 112.522) (end 141.478 114.046) (width 0.254) (layer F.Cu) (net 26))
+  (segment (start 145.1375 112.522) (end 143.002 112.522) (width 0.254) (layer F.Cu) (net 26))
   (segment (start 153.2655 121.285) (end 153.2655 119.38) (width 0.3048) (layer F.Cu) (net 31))
   (segment (start 153.151 119.2655) (end 153.2655 119.38) (width 0.3048) (layer F.Cu) (net 31))
@@
   (segment (start 152.7594 97.4325) (end 152.527 97.6649) (width 0.254) (layer F.Cu) (net 34))
   (segment (start 154.686 97.4325) (end 152.7594 97.4325) (width 0.254) (layer F.Cu) (net 34))
+  (segment (start 146.9625 112.522) (end 146.9625 112.3715) (width 0.254) (layer F.Cu) (net 35))
+  (segment (start 147.8965 111.4375) (end 148.601 111.4375) (width 0.254) (layer F.Cu) (net 35))
+  (segment (start 146.9625 112.3715) (end 147.8965 111.4375) (width 0.254) (layer F.Cu) (net 35))
   (zone (net 1) (net_name GND) (layer In1.Cu) (hatch edge 0.508)
     (connect_pads yes (clearance 0.508))
